File: SyncFix64.kicad_pcb (KiCad board)
At the start: 2 copper layers, 27.9 x 12.7 mm, 18 parts, among them J1 PWR, J2 Video, Q1 BSS138, Q2 BSS138, U1 LM1881, U2 AMS1117-50

Commit message: Layout improvements.
Parts:
- added J3: AltPwr, Pin_Headers:Pin_Header_Straight_1x01_Pitch2.54mm, F.Cu at (146.1, 74.9)
- added REF**: VIA-0.6mm, hackup:VIA-0.6mm, F.Cu at (141.9, 70.2)
- J1: value PWR -> Pwr; footprint Pin_Headers:Pin_Header_Angled_1x02_Pitch2.54mm -> Pin_Headers:Pin_Header_Straight_1x02_Pitch2.54mm
- J2: footprint Pin_Headers:Pin_Header_Angled_1x03_Pitch2.54mm -> Pin_Headers:Pin_Header_Straight_1x03_Pitch2.54mm
- moved J1 1.84 mm to (145.9, 67.6)
- moved J2 1.71 mm to (118.3, 77.5)
Routing:
- net +12V: track 10.1 -> 13.8 mm
- net VideoOUT: track 25.2 -> 28.8 mm, vias 0 -> 1
- net GND: track 11.8 -> 9.16 mm
- net +5V: track 30.4 -> 32.5 mm
- net VideoIN: track 4.77 -> 5.55 mm
Other:
- board size 27.9 x 12.7 mm -> 30.5 x 12.7 mm
- board text added: "12V"
- board text added: "5V"
- board text added: "GND"
- board text added: "IN"
- board text added: "OUT"
- board text added: "SyncFix64 v1.0"
- board text added: "github.com/hackup/SyncFix64"
