File: SyncFix64.kicad_pcb (KiCad board)
At the start: 2 copper layers, 30.5 x 12.7 mm, 20 parts, among them J1 Pwr, J2 Video, J3 AltPwr, Q1 BSS138, Q2 BSS138, U1 LM1881, U2 AMS1117-50

Commit message: Updates for version 1.1.
Parts:
- removed R4: 1M, Resistors_SMD:R_0805_HandSoldering
- removed REF** (x4): VIA-0.6mm, hackup:VIA-0.6mm
- R1: value 220 -> 100
- moved C5 0.70 mm to (134.3, 75.4)
- moved U2 0.51 mm to (140.3, 74.9)
- moved C1 0.44 mm to (133.5, 71.5)
- moved C3 0.44 mm to (133.5, 67.4)
- moved R2 0.36 mm to (133.6, 69.5)
- moved Q2 0.32 mm to (129.4, 75.4)
- moved C4 0.13 mm to (140.0, 67.8)
- moved J3 0.13 mm to (145.9, 74.9)
- moved U1 0.13 mm to (127.1, 69.3)
Routing:
- net GND: track 9.16 -> 0.00 mm, vias 0 -> 5
- net VideoOUT: track 28.8 -> 24.7 mm
- net +12V: track 13.8 -> 12.0 mm
- net +5V: track 32.5 -> 31.1 mm
- net Net-(Q1-Pad1): track 5.80 -> 6.53 mm
Other:
- board text added: "SyncFix64 v1.1"
- board text removed: "SyncFix64 v1.0"
