File: SyncFix64.kicad_pcb (KiCad board)
At the start: 2 copper layers, 30.5 x 12.7 mm, 15 parts, among them J1 Pwr, J2 Video, J3 AltPwr, Q1 BSS138, Q2 BSS138, U1 LM1881, U2 AMS1117-50

Commit message: Added logo.
Parts:
- added G***: LOGO, Logo:bigby, B.Cu at (124.7, 70.6)

Commit message: Version increment.
Other:
- board text added: "SyncFix64 v1.2"
- board text removed: "SyncFix64 v1.1"
Changed lines of the file:
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@@
-(kicad_pcb (version 20171130) (host pcbnew "(2017-12-18 revision 3c6d17026)-makepkg")
+(kicad_pcb (version 20171130) (host pcbnew "(5.0.0-rc2-dev-493-gd776eaca8)")
   (general
     (thickness 1.6)
@@
   (title_block
     (title SyncFix64)
-    (date 2018-01-01)
-    (rev 1.1)
+    (date 2018-05-28)
+    (rev 1.2)
     (company hackup.net)
   )
@@
     (at 124.714 70.612 180)
     (fp_text reference G*** (at 0 0 180) (layer B.SilkS) hide
-      (effects (font (thickness 0.3)) (justify mirror))
+      (effects (font (size 1.524 1.524) (thickness 0.3)) (justify mirror))
     )
     (fp_text value LOGO (at 0.75 0 180) (layer B.SilkS) hide
-      (effects (font (thickness 0.3)) (justify mirror))
+      (effects (font (size 1.524 1.524) (thickness 0.3)) (justify mirror))
     )
     (fp_poly (pts (xy -0.255603 2.783367) (xy -0.191997 2.7829) (xy -0.131892 2.782028) (xy -0.076809 2.780753)
@@
       (xy -0.452223 2.782322) (xy -0.387237 2.783079) (xy -0.32119 2.783427) (xy -0.255603 2.783367)) (layer B.SilkS) (width 0.01))
   )
-  (gr_text 5V (at 146.558 76.835 90) (layer F.SilkS)
+  (gr_text 5V (at 146.05 76.708) (layer F.SilkS)
     (effects (font (size 0.8 0.8) (thickness 0.15)))
   )
-  (gr_text "SyncFix64 v1.1" (at 136.017 73.406) (layer B.SilkS)
+  (gr_text "SyncFix64 v1.2" (at 136.017 73.406) (layer B.SilkS)
     (effects (font (size 1.5 1.5) (thickness 0.3)) (justify mirror))
   )
