File: SyncFix64.sch (KiCad schematic (older format))
At the start: 16 parts, among them J1 Pwr, J2 Video, J3 AltPwr, Q1 BSS138, Q2 BSS138, U1 LM1881, U2 AMS1117-50

Commit message: Updates for version 1.1.
Parts:
- removed R4: 1M, Resistors_SMD:R_0805_HandSoldering, symbol device:R
- R1: value 220 -> 100
Connections:
- wire segments 41 -> 40
Changed lines of the file:
@@
 Sheet 1 1
 Title "SyncFix64"
-Date "2017-12-29"
-Rev "1.0"
+Date "2018-01-01"
+Rev "1.1"
 Comp "hackup.net"
 Comment1 ""
@@
 $EndComp
 $Comp
-L device:R R4
-U 1 1 5A457088
-P 6650 2300
-F 0 "R4" H 6720 2346 50  0000 L CNN
-F 1 "1M" H 6720 2255 50  0000 L CNN
-F 2 "Resistors_SMD:R_0805_HandSoldering" V 6580 2300 50  0001 C CNN
-F 3 "" H 6650 2300 50  0001 C CNN
-	1    6650 2300
-	1    0    0    -1
-$EndComp
-$Comp
 L power:+5V #PWR08
 U 1 1 5A45711B
@@
 $EndComp
 $Comp
-L power:+5V #PWR09
-U 1 1 5A457145
-P 6650 2150
-F 0 "#PWR09" H 6650 2000 50  0001 C CNN
-F 1 "+5V" H 6665 2323 50  0000 C CNN
-F 2 "" H 6650 2150 50  0001 C CNN
-F 3 "" H 6650 2150 50  0001 C CNN
-	1    6650 2150
-	1    0    0    -1
-$EndComp
-$Comp
 L power:GND #PWR010
 U 1 1 5A4583C6
@@
 P 3000 2650
 F 0 "R1" H 3070 2696 50  0000 L CNN
-F 1 "220" H 3070 2605 50  0000 L CNN
+F 1 "100" H 3070 2605 50  0000 L CNN
 F 2 "Resistors_SMD:R_0805_HandSoldering" V 2930 2650 50  0001 C CNN
 F 3 "" H 3000 2650 50  0001 C CNN
@@
 VideoOUT
 Wire Wire Line
-	6650 2450 6650 2500
-Wire Wire Line
 	5850 2450 5850 2500
 Wire Wire Line
@@
 Wire Wire Line
 	7100 3950 7200 3950
-Connection ~ 6650 2500
 Wire Wire Line
 	6650 2500 6650 2550
